File: ErgoW-main.kicad_pcb (KiCad board)
At the start: 2 copper layers, 24.9 x 37 mm, 31 parts, among them J1 USB_C_Receptacle_USB2.0_16P, J2 Conn_01x03_Pin, J3 Conn_01x33_Socket, U2 XC6220B331MR, U3 BQ24075RGT, X1 32768kHz

Commit message: refactor: debug 3pin->4pin
Parts:
- J2: value Conn_01x03_Pin -> Conn_01x04_Pin; footprint Connector_PinHeader_1.00mm:PinHeader_1x03_P1.00mm_Vertical -> Connector_PinHeader_1.00mm:PinHeader_1x04_P1.00mm_Vertical
- moved J2 1.15 mm to (138.9, 110.4)
Connections:
- J2 pad 1: GND -> nRF_VDD
- J2 pad 2: SWD -> GND
- J2 pad 3: SWC -> SWD
Routing:
- net nRF_VDD: track 0.00 -> 52.2 mm, vias 0 -> 2
