File: ErgoW-main.kicad_sch (KiCad schematic)
At the start: 31 parts, among them J1 USB_C_Receptacle_USB2.0_16P, J2 Conn_01x03_Pin, J3 Conn_01x33_Socket, U2 XC6220B331MR, U3 BQ24075RGT, X1 32768kHz

Commit message: refactor: debug 3pin->4pin
Parts:
- J2: value Conn_01x03_Pin -> Conn_01x04_Pin; footprint Connector_PinHeader_1.00mm:PinHeader_1x03_P1.00mm_Vertical -> Connector_PinHeader_1.00mm:PinHeader_1x04_P1.00mm_Vertical; symbol Connector_Generic:Conn_01x03 -> Connector_Generic:Conn_01x04
Connections:
- net GND: now also J2.2 (Pin_2); no longer J2.1 (Pin_1)
- net SWC: now also J2.4 (Pin_4); no longer J2.3 (Pin_3)
- net SWD: now also J2.3 (Pin_3); no longer J2.2 (Pin_2)
- net nRF_VDD: now also J2.1 (Pin_1)
Changed lines of the file:
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@@
 		)
 	)
+	(global_label "nRF_VDD"
+		(shape input)
+		(at 201.93 46.99 180)
+		(fields_autoplaced yes)
+		(effects
+			(font
+				(size 1.27 1.27)
+			)
+			(justify right)
+		)
+		(property "Intersheetrefs" "${INTERSHEET_REFS}"
+			(at 190.841 46.99 0)
+			(effects
+				(font
+					(size 1.27 1.27)
+				)
+				(justify right)
+				(hide yes)
+			)
+		)
+	)
 	(global_label "P0.20"
 		(shape input)
@@
 	)
 	(symbol
-		(lib_id "Connector_Generic:Conn_01x03")
-		(at 207.01 52.07 0)
+		(lib_id "Connector_Generic:Conn_01x04")
+		(at 207.01 49.53 0)
 		(unit 1)
 		(exclude_from_sim no)
@@
 		(dnp no)
 		(property "Reference" "J2"
-			(at 211.582 54.102 0)
+			(at 211.582 51.562 0)
 			(effects
 				(font
@@
 			)
 		)
-		(property "Value" "Conn_01x03_Pin"
-			(at 224.536 51.308 0)
+		(property "Value" "Conn_01x04_Pin"
+			(at 224.536 48.768 0)
 			(effects
 				(font
@@
 			)
 		)
-		(property "Footprint" "Connector_PinHeader_1.00mm:PinHeader_1x03_P1.00mm_Vertical"
-			(at 207.01 52.07 0)
+		(property "Footprint" "Connector_PinHeader_1.00mm:PinHeader_1x04_P1.00mm_Vertical"
+			(at 207.01 49.53 0)
 			(effects
 				(font
@@
 		)
 		(property "Datasheet" "~"
-			(at 207.01 52.07 0)
+			(at 207.01 49.53 0)
 			(effects
 				(font
@@
 			)
 		)
-		(property "Description" "Generic connector, single row, 01x03, script generated (kicad-library-utils/schlib/autogen/connector/)"
-			(at 207.01 52.07 0)
+		(property "Description" "Generic connector, single row, 01x04, script generated (kicad-library-utils/schlib/autogen/connector/)"
+			(at 207.01 49.53 0)
 			(effects
 				(font
@@
 		(pin "3"
 		)
+		(pin "4"
+		)
 		(instances
-			(project ""
+			(project "ErgoW-main"
 				(path "/00177f65-620e-4f66-9d81-96167ce7d82d"
 					(reference "J2")
